File: ergogen-outputs/prime.kicad_pcb (KiCad board)
At the start: 2 copper layers, 313.6 x 138.6 mm, 84 parts

Commit message: Change board shape
Parts:
- moved D21 13.2 mm to (103.0, 73.4)
- moved D42 13.2 mm to (182.3, 73.4)
- moved D28 13.2 mm to (243.7, 4.78)
- moved D7 13.2 mm to (41.6, 4.78)
- moved D29 13.2 mm to (237.2, -13.1)
- moved D30 13.2 mm to (230.7, -30.9)
- moved D8 13.2 mm to (48.1, -13.1)
- moved D9 13.2 mm to (54.6, -30.9)
- moved D20 13.2 mm to (89.8, 55.9)
- moved D41 13.2 mm to (195.5, 55.9)
- moved D10 13.2 mm to (62.1, 6.23)
- moved D11 13.2 mm to (69.2, -11.4)
- moved D31 13.2 mm to (223.2, 6.23)
- moved D32 13.2 mm to (216.1, -11.4)
- moved D12 13.2 mm to (76.3, -29.0)
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Other:
- board size 313.6 x 138.6 mm -> 314.7 x 144.5 mm
