File: matrix.kicad_sch (KiCad schematic)
At the start: 84 parts

Commit message: first jlc submission
Parts:
- S1: LCSC (none) -> C5333465
Changed lines of the file:
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@@
       (effects (font (size 1.27 1.27)))
+    )
+    (property "LCSC" "C5333465" (at 59.69 50.8 0)
+      (effects (font (size 1.27 1.27)) hide)
     )
     (pin "2")
